File: filter_actuator_rev1.kicad_pcb (KiCad board)
At the start: 4 copper layers, 80 x 40 mm, 91 parts, among them J3 USB-C (2.0), J4 IPL1-102-01-F-S-RA-K, J5 IPL1-104-01-F-S-RA-K, U1 TPS561300DDCR, U2 STM32F042, U3 CP2102C, U4 MP6602, Y1 24 MHz XO

Commit message: Doing a commit because laptop is about to crash
Parts:
- C20, C22: footprint techne_capacitors:C_0805_2012Metric -> techne_capacitors:C_0402_1005Metric
- moved C26 63.1 mm to (67.3, 83.0), turned to 90 degrees
- moved R23 60.4 mm to (66.3, 83.0), turned to -90 degrees
- moved R2 58.2 mm to (124.7, 102.2), turned to 180 degrees
- moved C6 58.2 mm to (126.6, 102.2)
- moved R3 56.7 mm to (122.7, 102.2), turned to 180 degrees
- moved U1 54.8 mm to (124.2, 99.6), turned to -90 degrees
- moved C5 52.9 mm to (121.5, 99.2), turned to -90 degrees
- moved C4 51.9 mm to (119.3, 99.8), turned to -90 degrees
- moved L1 50.9 mm to (127.6, 93.6), turned to 90 degrees
- moved J1 48.8 mm to (110.2, 97.1), turned to 90 degrees
- moved C2 44.4 mm to (116.8, 99.8), turned to -90 degrees
- moved J2 43.7 mm to (68.8, 76.7), turned to 180 degrees
- moved C11 39.4 mm to (121.8, 92.6), turned to -90 degrees
- moved B1 38.2 mm to (71.9, 81.4)
- moved D1 32.3 mm to (69.2, 68.5)
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Connections:
- B2 pad 4: /BUT_POS1 -> /BUT_POS4
- B3 pad 4: /BUT_POS2 -> /BUT_POS3
- B4 pad 4: /BUT_POS3 -> /BUT_POS2
- B5 pad 4: /BUT_POS4 -> /BUT_POS1
- C27 pad 1: /BUT_POS1 -> /BUT_POS4
- C28 pad 1: /BUT_POS2 -> /BUT_POS3
- C29 pad 1: /BUT_POS3 -> /BUT_POS2
- C30 pad 1: /BUT_POS4 -> /BUT_POS1
- D2 pad K: /POS1 -> /POS4
- D3 pad K: /POS2 -> /POS3
- D4 pad K: /POS3 -> /POS2
- D5 pad K: /POS4 -> /POS1
- R24 pad 2: /BUT_POS1 -> /BUT_POS4
- R25 pad 2: /BUT_POS2 -> /BUT_POS3
- R26 pad 2: /BUT_POS3 -> /BUT_POS2
- R27 pad 2: /BUT_POS4 -> /BUT_POS1
- U2 pad 10: /MP6602_nRST -> unconnected-(U2-PA0-Pad10)
- U2 pad 11: /MP6602_SLEEP -> unconnected-(U2-PA1-Pad11)
- U2 pad 20: /BUT_POS2 -> /BUT_POS1
- U2 pad 21: /POS1 -> /MP6602_ENBL
- U2 pad 22: /POS2 -> /MP6602_nFAULT
- U2 pad 25: /POS3 -> /MP6602_nRST
- U2 pad 26: /POS4 -> /MP6602_SLEEP
- U2 pad 27: /BUT_POS1 -> /POS1
- U2 pad 28: /MP6602_nFAULT -> /BUT_POS2
- U2 pad 29: /ENC_CHB -> /POS2
- U2 pad 30: /ENC_CHA -> /BUT_POS3
- U2 pad 31: unconnected-(U2-PA10,TIM1_CH3-Pad31) -> /POS3
- U2 pad 38: /MP6602_ENBL -> /BUT_POS4
- U2 pad 39: /LIM_A -> /POS4
- U2 pad 45: /BUT_POS4 -> unconnected-(U2-PB8,CAN_RX-Pad45)
- U2 pad 46: /BUT_POS3 -> unconnected-(U2-PB9,CAN_RX-Pad46)
Routing:
- net /CS: track 0.00 -> 58.3 mm, vias 0 -> 1
- net /SCLK: track 0.00 -> 57.2 mm, vias 0 -> 1
- net /MISO: track 0.00 -> 55.0 mm, vias 0 -> 1
- net /MOSI: track 0.00 -> 53.9 mm, vias 0 -> 1
- net /STEP: track 0.00 -> 51.3 mm, vias 0 -> 1
- net /DIR: track 0.00 -> 49.3 mm, vias 0 -> 1
- net /MP6602_nRST: track 0.00 -> 44.0 mm, vias 0 -> 1
- net /MP6602_nFAULT: track 0.00 -> 40.2 mm, vias 0 -> 1
- net /MP6602_ENBL: track 0.00 -> 39.2 mm, vias 0 -> 1
- net /BUT_POS1: track 1.37 -> 40.3 mm
- net GND: track 0.00 -> 2.46 mm, vias 0 -> 11
- net +3.3V: track 0.00 -> 2.38 mm, vias 0 -> 21
- net /POS1: track 0.00 -> 2.31 mm
- net Net-(U4-VG): track 0.00 -> 1.33 mm
- net /MP6602_SLEEP: track 0.00 -> 1.28 mm, vias 0 -> 1
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- added copper zone on F.Cu, net +12V
- added copper zone on F.Cu, net +3.3V
- added copper zone on F.Cu, net /AOUT1
- added copper zone on F.Cu, net /BOUT1
- added copper zone on F.Cu, net /BOUT2

Commit message: Initial layout complete. Need to review before ordering.
Parts:
- removed R12, R13, R14: 10K, resistors:R_0402_1005Metric
- C14, C15, R1: moved to B.Cu
- moved C1 23.4 mm to (67.5, 73.8), turned to 90 degrees
- moved R4 11.7 mm to (67.6, 93.0), turned to 180 degrees
- moved C10 9.29 mm to (69.6, 97.3), turned to -90 degrees
- moved R18 9.16 mm to (102.4, 94.9), turned to 0 degrees
- moved R23 9.11 mm to (62.2, 91.1), turned to 0 degrees
- moved C26 8.73 mm to (62.2, 90.1), turned to 180 degrees
- moved B1 8.21 mm to (71.1, 73.2)
- moved R11 8.19 mm to (94.1, 96.0), turned to 180 degrees
- moved C15 8.06 mm to (99.5, 98.2), turned to -90 degrees
- moved R16 7.81 mm to (83.4, 88.7), turned to 90 degrees
- moved R17 7.70 mm to (78.8, 85.6), turned to 0 degrees
- moved C14 7.21 mm to (100.7, 96.7), turned to 0 degrees
- moved R22 6.82 mm to (84.4, 88.7), turned to -90 degrees
- moved C8 6.52 mm to (68.5, 88.0), turned to 180 degrees
- moved R1 6.48 mm to (66.5, 73.8), turned to -90 degrees
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Connections:
- U2 pad 11: unconnected-(U2-PA1-Pad11) -> /CP_nRST
- U2 pad 2: /LMT_SW -> unconnected-(U2-PC13-Pad2)
- U2 pad 32: /USB_D- -> unconnected-(U2-PA11,USB_DM-Pad32)
- U2 pad 33: /USB_D+ -> unconnected-(U2-PA12,USB_DP-Pad33)
- U2 pad 40: /LIM_B -> /LMT_SW
- U2 pad 41: /CP_nRST -> unconnected-(U2-PB5-Pad41)
Routing:
- net GND: track 2.46 -> 57.1 mm, vias 11 -> 113
- net /POS1: track 2.31 -> 52.3 mm, vias 0 -> 1
- net /MP6602_SLEEP: track 1.28 -> 49.8 mm, vias 1 -> 3
- net /POS2: track 0.00 -> 44.1 mm, vias 0 -> 1
- net /POS3: track 0.00 -> 35.2 mm, vias 0 -> 1
- net +3.3V: track 2.38 -> 36.8 mm, vias 21 -> 47
- net /BUT_POS2: track 1.37 -> 33.3 mm
- net /POS4: track 0.00 -> 31.7 mm, vias 0 -> 3
- net /nRST: track 0.00 -> 29.7 mm, vias 0 -> 3
- net /CP_nRST: track 0.00 -> 29.6 mm, vias 0 -> 2
- net /BUT_POS3: track 1.37 -> 25.9 mm, vias 0 -> 1
- net /BUT_POS4: track 1.37 -> 23.5 mm, vias 0 -> 3
- net /CP_RXD: track 0.00 -> 21.4 mm, vias 0 -> 2
- net /CP_TXD: track 0.00 -> 20.3 mm
- net /LMT_SW: track 0.00 -> 16.1 mm
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- added copper zone on In2.Cu, net +12V
- added copper zone on B.Cu, net GND
- added copper zone on F.Cu, net GND
- added copper zone on F.Cu, net Net-(U1-SW)
Other:
- board text added: "LMT SW"
- board text added: "Luxel Filter Actuator Rev 1.0"
- board text added: "MOTOR"
- board text added: "POS1"
- board text added: "POS2"
- board text added: "POS3"
- board text added: "POS4"
- board text added: "POWER"

Commit message: Tag as ordered for fab from JLC. Official Rev1
Parts:
- moved F2 8.10 mm to (112.3, 101.7)
Routing:
- net +3.3V: track 36.8 -> 37.5 mm
