File: filter_actuator_rev1.kicad_sch (KiCad schematic)
At the start: 0 parts

Commit message: First push to get schematic ready
Parts:
- added B1, B2, B4, B5: (no value), techne_mechanical:B3FS-1032, symbol techne_mechanical:B3FS-1052
- added B3: (no value), techne_mechanical:C&K_pushbutton, symbol techne_mechanical:smd_button
- added C1, C2, C3, C6, C7: 22uF, techne_capacitors:C_1812_4532Metric, symbol techne_capacitors:C_1812_4532Metric
- added C13, C17, C18: 1uF, techne_capacitors:C_0402_1005Metric, symbol techne_capacitors:C_0402_1005Metric
- added C19, C20, C21, C22, C24, C25: 0.1uF, techne_capacitors:C_0402_1005Metric, symbol techne_capacitors:C_0402_1005Metric
- added C4, C5: 10uF, techne_capacitors:C_1206_3216Metric, symbol techne_capacitors:C_1206_3216Metric
- added C8, C9: 1uF, techne_capacitors:C_0805_2012Metric, symbol techne_capacitors:C_0805_2012Metric
- added D1, D2, D3, D4: GRN, techne_diodes:LIteOn_0603, symbol techne_diodes:LiteOn_LED_GRN
- added D5: RED, techne_diodes:LIteOn_0603, symbol techne_diodes:LiteOn_LED_RED
- added J1: (no value), techne_connectors:PJ-002AH_Power Barrel, symbol techne_connectors:PJ-002AH
- added J2: IPL1-106-01-F-S-RA-K, techne_connectors:SAMTEC_IPL1-106-01-X-S-RA-K, symbol techne_connectors:IPL1-106-01-F-S-RA-K
- added J3: QT04ASB83H0000G, techne_connectors:Anytek_wire2brd_4pos, symbol techne_connectors:wire2board_4pin
- added J5: (no value), JLink:JLink_needle_6pin, symbol prog_debug:JLink_Needle_6pin
- added J7: N/A, techne_connectors:PinHeader_1x04_P2.54mm_Vertical, symbol techne_connectors:1x4_header, 0.1{dblquote} pitch
- added LP1, LP2, LP3, LP4, LP5: 0.25in, techne_mechanical:Dialight_515-1314-xxxx, symbol techne_mechanical:Lightpipe_0.25in
- added R1, R15, R16, R17, R2, R25, R3, R4, R5, R7: 1K, resistors:R_0402_1005Metric, symbol resistors:R_0402_1005Metric
- added R10, R20, R21: 10K, resistors:R_0402_1005Metric, symbol resistors:R_0402_1005Metric
- added U2: MP6602, techne_motordrivers:QFN-25_MP6602_MNP, symbol techne_motordrivers:MP6602
- added U3: STM32F042, techne_qfpn:QFN50P700X700X60-49N, symbol techne_stmicro:STM32F042C6U
- added Y1: 24 MHz XO, techne_osc_clks:OSC_ECS-2333-480-BN-TR, symbol techne_osc_clks:ECS_48MHz_XO
Connections:
- new net: J1.2 (GND), J1.3 (GND)
- new net: R17.2, U2.9 (ENBL)
- new net: C18.1, U2.11 (VG)
- new net: C17.1, U2.12 (VCP)
- new net: J3.1, U2.4 (AOUT2)
- new net: R15.2, U2.6 (SLEEP)
- new net: R16.2, U2.7 (nRESET)
- new net: R20.1, U3.44 (PF11-BOOT0)
- new net: J7.2, U3.13 (PA3,USART2_RX)
- new net: J7.3, U3.12 (PA2,USART2_TX)
- new net: B1.1, B1.2
- new net: D5.A, R5.2
- new net: D2.A, R2.2
- new net: D1.A, R1.2
- new net: B4.1, B4.2
- new net: B5.1, B5.2
- new net: J5.2 (SWDIO), U3.34 (PA13,SWDIO)
- new net: J5.4 (SWCLK), U3.37 (PA14,SWCLK)
- new net: B2.1, B2.2
- new net: D4.A, R4.2
- new net: D3.A, R3.2
- new net: U3.5 (PF0_OSC_IN), Y1.3 (OUT)
- new net +12V: C1.1, C17.2, C2.1, C3.1, C4.1, C5.1, C6.1, C7.1, C8.1, C9.1, U2.15 (VIN), U2.3 (VIN)
- new net +3.3V: C13.1, C19.1, C20.1, C21.1, C22.1, C25.1, J5.1 (VTref), J7.1, R1.1, R15.1, R16.1, R17.1, R2.1, R21.1, R25.1, R3.1, R4.1, R5.1, R7.1, U2.21 (VCC), U3.1 (VBAT), U3.24 (VDD), U3.36 (VDDIO2), U3.48 (VDD), U3.9 (VDDA), Y1.1 (EN), Y1.4 (VDD)
- new net ACT_IN: U3.20 (PB2)
- new net ACT_OUT: U3.27 (PB14)
- new net AOUT1: J3.2, U2.2 (AOUT1)
- new net BOUT1: J3.3, U2.16 (BOUT1)
- new net BOUT2: J3.4, U2.14 (BOUT2)
- new net CS: U2.23 (nSCS), U3.14 (PA4,SP1_NSS)
- new net DIR: R7.2, U2.18 (DIR), U3.19 (PB1)
- new net ENC_CHA: U3.30 (PA9,TIM1_CH2)
- new net ENC_CHB: U3.29 (PA8,TIM1_CH1)
- new net ENC_IDX: U3.10 (PA0)
- new net GND: B3.1, B3.2, C1.2, C13.2, C18.2, C19.2, C2.2, C20.2, C21.2, C22.2, C24.2, C25.2, C3.2, C4.2, C5.2, C6.2, C7.2, C8.2, C9.2, D5.K, J5.5 (GND), J7.4, R10.2, R20.2, U2.1 (PGND), U2.10 (GND), U2.13 (PGND), U2.17 (PGND), U2.25 (PGND), U2.5 (PGND), U3.23 (VSS), U3.35 (VSS), U3.47 (VSS), U3.8 (VSSA), U3.EP (VSS), Y1.2 (GND)
- new net LIM_A: U3.39 (PB3)
- new net LIM_B: U3.40 (PB4)
- new net MISO: U2.20 (SDATO), U3.16 (PA6,SPI1_MISO)
- new net MOSI: U2.22 (SDATI), U3.17 (PA7,SPI1_MOSI)
- new net POS1: D1.K, U3.21 (PB10)
- new net POS2: D2.K, U3.22 (PB11)
- new net POS3: D3.K, U3.25 (PB12)
- new net POS4: D4.K, U3.26 (PB13)
- new net SCLK: U2.24 (SCLK), U3.15 (PA5,SPI1_SCK)
- new net STEP: R10.1, U2.19 (STEP), U3.18 (PB0,TIM3_CH3)
- new net USB_D+: U3.33 (PA12,USB_DP)
- new net USB_D-: U3.32 (PA11,USB_DM)
- new net USB_REN: U3.38 (PA15)
- new net nFAULT: R25.2, U2.8 (nFAULT), U3.28 (PB15)
- new net nRST: B3.4, C24.1, J5.3 (nRESET), R21.2, U3.7 (NRST)
- no-connect marks 0 -> 1
Other:
- note added: "Button: B3FS-1052 Cap: B32-2000 Figure out distance between enclosure and board"
- note added: "Layout Cover EP under MP6602 with GND vias GND Pour on 1st layer under part and in between motor coil connections"
- note added: "TPS561300DDCR - 12V to 3.3V, 1 A buck"
- company: (none) -> Techne Solutions, LLC
- title: (none) -> Luxel Filter Actuator Motor Drive Board

Commit message: Finished part placement. Waiting on some feedback from Patrick on connector and interface placement.
Parts:
- removed J2: IPL1-106-01-F-S-RA-K, techne_connectors:SAMTEC_IPL1-106-01-X-S-RA-K, symbol techne_connectors:IPL1-106-01-F-S-RA-K
- removed J3: QT04ASB83H0000G, techne_connectors:Anytek_wire2brd_4pos, symbol techne_connectors:wire2board_4pin
- removed J7: N/A, techne_connectors:PinHeader_1x04_P2.54mm_Vertical, symbol techne_connectors:1x4_header, 0.1{dblquote} pitch
- added C11: 22uF, techne_capacitors:C_1812_4532Metric, symbol techne_capacitors:C_1812_4532Metric
- added C14: 4.7uF, techne_capacitors:C_0402_1005Metric, symbol techne_capacitors:C_0402_1005Metric
- added C15, C26, C27, C28, C29, C30: 0.1uF, techne_capacitors:C_0402_1005Metric, symbol techne_capacitors:C_0402_1005Metric
- added C2, C4: 10uF, techne_capacitors:C_1206_3216Metric, symbol techne_capacitors:C_1206_3216Metric
- added C5: 1uF, techne_capacitors:C_0805_2012Metric, symbol techne_capacitors:C_0805_2012Metric
- added C6: 56pF, techne_capacitors:C_0402_1005Metric, symbol techne_capacitors:C_0402_1005Metric
- added F1, F2, F3, F4: (no value), techne_mechanical:fiducial_1mm_2mm, symbol techne_mechanical:fiducial_1mm_2mm
- added J3: USB-C (2.0), techne_connectors:SAMESKY_UJ20-C-H-G-SMT-2A-P16-TR, symbol techne_connectors:USB-C_(USB2.0)
- added J4: IPL1-102-01-F-S-RA-K, techne_connectors:SAMTEC_IPL1-102-01-X-S-RA-K, symbol techne_connectors:IPL1-102-01-F-S-RA-K_1
- added J5: IPL1-104-01-F-S-RA-K, techne_connectors:SAMTEC_IPL1-104-01-X-S-RA-K, symbol techne_connectors:IPL1-104-01-F-S-RA-K
- added L1: 10uH, techne_inductors:IND_SRR6038-100Y, symbol techne_inductors:SRR6038
- added M1, M2, M3, M4: (no value), techne_mechanical:M3_NPLATED_TH, symbol techne_mechanical:M3_MountingHole
- added R10, R11: 5.1K, resistors:R_0402_1005Metric, symbol resistors:R_0402_1005Metric
- added R12, R13, R14, R18, R23, R24, R25, R26, R27: 10K, resistors:R_0402_1005Metric, symbol resistors:R_0402_1005Metric
- added R2: 100K, resistors:R_0402_1005Metric, symbol resistors:R_0402_1005Metric
- added R20: 1K, resistors:R_0402_1005Metric, symbol resistors:R_0402_1005Metric
- added R3: 22.1K, resistors:R_0402_1005Metric, symbol resistors:R_0402_1005Metric
- added U1: TPS561300DDCR, techne_ti_sot:ti_DDC0006A_SOT23, symbol techne_power:TPS561300
- added U3: CP2102C, techne_comms:IC_QFN24_SIL, symbol techne_comms:CP2102C
- renumbered B3 to B1, B1 to B2, B2 to B3, C24 to C1, C22 to C10, C1 to C12, C6 to C13, C13 to C16, C2 to C17, C7 to C18, C3 to C19, C8 to C20, C4 to C21, C9 to C22, C17 to C23, C18 to C24, C5 to C25, C25 to C3, C19 to C7, C20 to C8, C21 to C9, D5 to D1, D1 to D2, D2 to D3, D3 to D4, D4 to D5, J5 to J2, LP5 to LP1, LP1 to LP2, LP2 to LP3, LP3 to LP4, LP4 to LP5, R21 to R1, R25 to R15, R10 to R16, R15 to R17, R16 to R19, R17 to R21, R7 to R22, R20 to R4, R1 to R6, R2 to R7, R3 to R8, R4 to R9, U3 to U2, U2 to U4
Connections:
- net ACT_IN is gone; now on net BUT_POS2: U2.20 (PB2)
- net ACT_OUT is gone; now on net BUT_POS1: U2.27 (PB14)
- net ENC_IDX is gone; now on net MP6602_nRST: U2.10 (PA0)
- net USB_REN is gone; now on net MP6602_ENBL: U2.38 (PA15)
- net +12V: now also J1.1 (V+), C2.1, C4.1, C5.1, U1.3 (VIN)
- net +3.3V: now also C11.1, C14.1, C15.1, L1.2, R18.2, R2.1, R20.1, R23.1, R24.1, R25.1, R26.1, R27.1, U3.5 (VIO), U3.6 (VDD), U3.7 (VREGIN)
- net AOUT1: now also J5.2
- net BOUT1: now also J5.3
- net BOUT2: now also J5.4
- net GND: now also B2.1, B2.2, B3.1, B3.2, B4.1, B4.2, B5.1, B5.2, J1.2 (GND), J1.3 (GND), C11.2, C14.2, C15.2, C2.2, C26.2, C27.2, C28.2, C29.2, C30.2, C4.2, C5.2, J3.A1/B12 (GND), J3.B1/A12 (GND), J3.SH1 (GND), J3.SH2 (GND), J3.SH3 (GND), J3.SH4 (GND), J4.1, R10.2, R11.2, R13.2, R3.2, U1.1 (GND), U3.2 (GND), U3.EP (GND)
- net USB_D+: now also J3.A6 (Dp1), J3.B6 (Dp2), U3.3 (D+)
- net USB_D-: now also J3.A7 (Dn1), J3.B7 (Dn2), U3.4 (D-)
- net MP6602_ENBL: now reaches R21.2, U4.9 (ENBL)
- net AOUT2: now reaches U4.4 (AOUT2)
- net AOUT2: now also J5.1
- net MP6602_SLEEP: now reaches R17.2, U4.6 (SLEEP)
- net MP6602_SLEEP: now also U2.11 (PA1)
- net MP6602_nRST: now reaches R19.2, U4.7 (nRESET)
- net CP_TXD: now reaches U2.13 (PA3,USART2_RX)
- net CP_TXD: now also U3.21 (TXD)
- net CP_RXD: now reaches U2.12 (PA2,USART2_TX)
- net CP_RXD: now also U3.20 (RXD)
- net BUT_POS1: now reaches B2.4
- net BUT_POS1: now also C27.1, R24.2
- net BUT_POS3: now reaches B4.4
- net BUT_POS3: now also U2.46 (PB9,CAN_RX), C29.1, R26.2
- net BUT_POS4: now reaches B5.4
- net BUT_POS4: now also U2.45 (PB8,CAN_RX), C30.1, R27.2
- net BUT_POS2: now reaches B3.4
- net BUT_POS2: now also C28.1, R25.2
- net LMT_SW: now reaches U2.2 (PC13)
- net LMT_SW: now also C26.1, J4.2, R23.2
- net CP_nRST: now reaches U2.41 (PB5)
- net CP_nRST: now also R20.2, U3.9 (RSTb)
- net nFAULT renamed MP6602_nFAULT
- new net: R12.2, R13.1, R14.1
- new net: R14.2, R18.1, U3.8 (VBUS)
- new net: J3.A5 (CC1), R11.1
- new net: C6.2, L1.1, U1.2 (SW)
- new net: R2.2, R3.1, U1.4 (FB)
- new net: C6.1, U1.6 (BOOT)
- new net: J3.B5 (CC2), R10.1
- new net VBUS: J3.A4/B9 (VBUS), J3.B4/A9 (VBUS), R12.1
- no-connect marks 1 -> 12
Other:
- note added: "A 5V signal on the VBUS pin indicates a USB connection Tie to 3.3V with DNP resistor divider in case it doesn't work"
- note added: "BACK"
- note added: "FRONT"
- note removed: "Button: B3FS-1052 Cap: B32-2000 Figure out distance between enclosure and board"
- note removed: "TPS561300DDCR - 12V to 3.3V, 1 A buck"
- moved on the sheet: B2, B3, B4, B5, J1, R15, R17, R19, R21

Commit message: Doing a commit because laptop is about to crash
Parts:
- removed C20, C22: 1uF, techne_capacitors:C_0805_2012Metric, symbol techne_capacitors:C_0805_2012Metric
- added C20, C22: 1uF, techne_capacitors:C_0402_1005Metric, symbol techne_capacitors:C_0402_1005Metric
Connections:
- net ENC_CHA is gone; now on net BUT_POS3: U2.30 (PA9,TIM1_CH2)
- net ENC_CHB is gone; now on net POS2: U2.29 (PA8,TIM1_CH1)
- net LIM_A is gone; now on net POS4: U2.39 (PB3)
- net +12V: now also C20.1, C22.1
- net BUT_POS1: now also B5.4, C30.1, R27.2, U2.20 (PB2); no longer B2.4, C27.1, R24.2, U2.27 (PB14)
- net BUT_POS2: now also B4.4, C29.1, R26.2, U2.28 (PB15); no longer B3.4, C28.1, R25.2, U2.20 (PB2)
- net BUT_POS3: now also B3.4, C28.1, R25.2; no longer B4.4, C29.1, R26.2, U2.46 (PB9,CAN_RX)
- net BUT_POS4: now also B2.4, C27.1, R24.2, U2.38 (PA15); no longer B5.4, C30.1, R27.2, U2.45 (PB8,CAN_RX)
- net GND: now also C20.2, C22.2
- net MP6602_ENBL: now also U2.21 (PB10); no longer U2.38 (PA15)
- net MP6602_SLEEP: now also U2.26 (PB13); no longer U2.11 (PA1)
- net MP6602_nFAULT: now also U2.22 (PB11); no longer U2.28 (PB15)
- net MP6602_nRST: now also U2.25 (PB12); no longer U2.10 (PA0)
- net POS1: now also D5.K, U2.27 (PB14); no longer D2.K, U2.21 (PB10)
- net POS2: now also D4.K; no longer D3.K, U2.22 (PB11)
- net POS3: now also D3.K, U2.31 (PA10,TIM1_CH3); no longer D4.K, U2.25 (PB12)
- net POS4: now also D2.K; no longer D5.K, U2.26 (PB13)

Commit message: Initial layout complete. Need to review before ordering.
Parts:
- removed R12, R13, R14: 10K, resistors:R_0402_1005Metric, symbol resistors:R_0402_1005Metric
Connections:
- net LIM_B is gone; now on net LMT_SW: U2.40 (PB4)
- net CP_nRST: now also U2.11 (PA1); no longer U2.41 (PB5)
- net LMT_SW: no longer U2.2 (PC13)
- net USB_D+: no longer U2.33 (PA12,USB_DP)
- net USB_D-: no longer U2.32 (PA11,USB_DM)
- no-connect marks 12 -> 21

Commit message: Tag as ordered for fab from JLC. Official Rev1
Other:
- note added: "Input: 30V max input"
Changed lines of the file:
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@@
+		)
+	)
+	(text "Input: 30V max input"
+		(exclude_from_sim no)
+		(at 96.774 48.768 0)
+		(effects
+			(font
+				(size 1.27 1.27)
+			)
 		)
 	)
